File: kicad_v4/BagTag/BagTag.kicad_pcb (KiCad board)
At the start: 2 copper layers, 63.5 x 63.5 mm, 71 parts, among them J1 Conn_I2C, J10 Conn_01x03, J11 Conn_01x03, J12 Conn_01x03, J13 Conn_01x03, J14 Conn_01x03, J2 Conn_I2C, J20 D2, J21 D3, J22 D4, J23 D5, J24 D6, J25 D7, J26 D8, J27 D9, J28 D10, J29 D11, J3 Conn_01x03, J30 D12, J31 D13, J32 RST1, J33 RST1, J34 D0, J35 D1, J36 A7, J37 A6, J38 A5, J39 A4, J4 Conn_01x03, J40 A3, J41 A2, J42 A1, J43 A0, J44 AREF, J45 VIN, J46 5V, J47 3V3, J48 GND1, J49 GND2, J5 Conn_01x03, J6 Conn_01x03, J7 Conn_01x03, J8 Conn_01x03, J9 Conn_01x03, SW1 ON, U1 Arduino_Nano

Commit message: ver 4 WIP - gerbers are ready
Parts:
- removed kibuzzard-6461CA3D: G***, BagTag:kibuzzard-6461CA3D
- removed kibuzzard-663CECFE: G***, kibuzzard-663CECFE
- removed kibuzzard-663CED10: G***, kibuzzard-663CED10
- removed kibuzzard-663CED23: G***, kibuzzard-663CED23
- removed kibuzzard-663CED63: G***, kibuzzard-663CED63
- added kibuzzard-646134AD: G***, BagTag:kibuzzard-646134AD, B.Cu at (52.3, 92.7)
- added kibuzzard-646134AD: G***, BagTag:kibuzzard-646134AD, B.Cu at (84.1, 92.7)
- added kibuzzard-646134FF: G***, BagTag:kibuzzard-646134FF, B.Cu at (75.4, 92.7)
- added kibuzzard-646134FF: G***, BagTag:kibuzzard-646134FF, B.Cu at (107.2, 92.7)
- added kibuzzard-6640BED0: G***, kibuzzard-6640BED0, F.Cu at (66.0, 56.1)
- added kibuzzard-6640BED0: G***, kibuzzard-6640BED0, B.Cu at (66.0, 56.1)
- added kibuzzard-6640BEF1: G***, kibuzzard-6640BEF1, F.Cu at (94.0, 56.1)
- added kibuzzard-6640BEF1: G***, kibuzzard-6640BEF1, B.Cu at (94.0, 56.1)
- added kibuzzard-6640BF00: G***, kibuzzard-6640BF00, F.Cu at (101.3, 58.6)
- added kibuzzard-6640BF00: G***, kibuzzard-6640BF00, B.Cu at (101.3, 58.7)
- added kibuzzard-6640BF4C: G***, kibuzzard-6640BF4C, F.Cu at (106.7, 79.2)
- added kibuzzard-6640BF4C: G***, kibuzzard-6640BF4C, B.Cu at (106.7, 66.0)
- added kibuzzard-6640BFA2: G***, kibuzzard-6640BFA2, F.Cu at (66.0, 54.3)
- added kibuzzard-6640BFA2: G***, kibuzzard-6640BFA2, B.Cu at (66.0, 54.3)
- added kibuzzard-6640BFC5: G***, kibuzzard-6640BFC5, F.Cu at (94.0, 54.3)
- added kibuzzard-6640BFC5: G***, kibuzzard-6640BFC5, B.Cu at (94.0, 54.3)
- added kibuzzard-6640BFF1: G***, kibuzzard-6640BFF1, F.Cu at (103.1, 58.6)
- added kibuzzard-6640BFF1: G***, kibuzzard-6640BFF1, B.Cu at (103.2, 58.7)
- added kibuzzard-6640C3B8: G***, kibuzzard-6640C3B8, F.Cu at (100.6, 72.6)
- added kibuzzard-6640C3B8: G***, kibuzzard-6640C3B8, B.Cu at (100.5, 72.6)
- added kibuzzard-6640C421: G***, kibuzzard-6640C421, F.Cu at (59.7, 49.5)
- added kibuzzard-6640C421: G***, kibuzzard-6640C421, F.Cu at (87.6, 49.6)
- added kibuzzard-6640C44A: G***, kibuzzard-6640C44A, F.Cu at (108.0, 65.0)
- added kibuzzard-66412AF8: G***, kibuzzard-66412AF8, B.Cu at (50.3, 68.6)
- LED1: footprint BagTag:LED_matrix_8x8_M1088ASR -> BagTag:LED_8x8_M1088ASR
- moved kibuzzard-64612FED 31.0 mm to (49.3, 53.3), turned to 90 degrees (x2)
- moved kibuzzard-64612FA6 25.0 mm to (49.3, 60.5), turned to 90 degrees (x2)
- moved BT1 24.4 mm to (50.0, 58.2), turned to 180 degrees
- moved G*** 12.2 mm to (100.3, 81.0)
- moved D1 8.23 mm to (60.2, 79.0), turned to 180 degrees
- moved kibuzzard-6461377A 3.06 mm to (78.0, 63.8)
- moved kibuzzard-6461376B 3.06 mm to (78.0, 67.8)
- moved J28 3.05 mm to (65.3, 61.0)
- moved J44 3.05 mm to (65.3, 71.1)
- moved J20 3.05 mm to (85.6, 61.0)
- moved J21 3.05 mm to (83.1, 61.0)
- moved J22 3.05 mm to (80.5, 61.0)
- moved J24 3.05 mm to (75.4, 61.0)
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Connections:
- LED2 pad DIN: /MISO -> /DOUT
- LED2 pad DOUT: /DOUT -> unconnected-(LED2-PadDOUT)
Routing:
- net /GND: track 91.4 -> 248.6 mm
- net /MISO: track 76.1 -> 56.7 mm
- net /DOUT: track 32.8 -> 15.9 mm
- net /9V: track 5.96 -> 21.5 mm
- net /D10: track 108.0 -> 104.3 mm
- net /D6: track 27.0 -> 23.9 mm
- net /D9: track 32.1 -> 29.0 mm
- net /D3: track 24.5 -> 21.5 mm
- net /D5: track 27.1 -> 24.0 mm
- net /8V3: track 18.2 -> 20.5 mm
- net /A3: track 39.0 -> 36.8 mm
- net /D4: track 18.0 -> 20.0 mm
- net /MOSI: track 108.5 -> 106.6 mm
- net /D7: track 13.1 -> 14.9 mm
- net /D2: track 20.7 -> 22.6 mm
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Other:
- outline, holes or cut-outs redrawn
