File: hardware_PCB/TheThing_v7/TheThing_addon.kicad_pcb (KiCad board)
At the start: 2 copper layers, 75.2 x 29.6 mm, 44 parts, among them J15 HC-SR04, J16 Conn_01x10, Q1 PN2222ABU, SW2 ON, SW3 ON

Commit message: v7 prototype files for PCB and enclosure
Parts:
- moved kibuzzard-67A22DCA 5.30 mm to (41.3, 130.8)
- moved kibuzzard-67A22DE4 1.90 mm to (95.3, 130.8)
Changed lines of the file:
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@@
 	(footprint "kibuzzard-67A22DCA"
 		(layer "F.Cu")
-		(at 46.6 130.8)
+		(at 41.3 130.8)
 		(descr "Generated with KiBuzzard")
 		(tags "kb_params=eyJBbGlnbm1lbnRDaG9pY2UiOiAiQ2VudGVyIiwgIkNhcExlZnRDaG9pY2UiOiAiWyIsICJDYXBSaWdodENob2ljZSI6ICJdIiwgIkZvbnRDb21ib0JveCI6ICJVYnVudHVNb25vLUIiLCAiSGVpZ2h0Q3RybCI6IDEuMCwgIkxheWVyQ29tYm9Cb3giOiAiRi5TaWxrUyIsICJMaW5lU3BhY2luZ0N0cmwiOiAxLjgsICJNdWx0aUxpbmVUZXh0IjogIlNXSVRDSCIsICJQYWRkaW5nQm90dG9tQ3RybCI6IDIuMCwgIlBhZGRpbmdMZWZ0Q3RybCI6IDIuMCwgIlBhZGRpbmdSaWdodEN0cmwiOiAyLjAsICJQYWRkaW5nVG9wQ3RybCI6IDIuMCwgIldpZHRoQ3RybCI6IDEuMywgImFkdmFuY2VkQ2hlY2tib3giOiBmYWxzZSwgImlubGluZUZvcm1hdFRleHRib3giOiBmYWxzZSwgImxpbmVvdmVyU3R5bGVDaG9pY2UiOiAiU3F1YXJlIiwgImxpbmVvdmVyVGhpY2tuZXNzQ3RybCI6IDF9")
@@
 	(footprint "kibuzzard-67A22DE4"
 		(layer "F.Cu")
-		(at 93.4 130.8)
+		(at 95.3 130.8)
 		(descr "Generated with KiBuzzard")
 		(tags "kb_params=eyJBbGlnbm1lbnRDaG9pY2UiOiAiQ2VudGVyIiwgIkNhcExlZnRDaG9pY2UiOiAiWyIsICJDYXBSaWdodENob2ljZSI6ICJdIiwgIkZvbnRDb21ib0JveCI6ICJVYnVudHVNb25vLUIiLCAiSGVpZ2h0Q3RybCI6IDEuMCwgIkxheWVyQ29tYm9Cb3giOiAiRi5TaWxrUyIsICJMaW5lU3BhY2luZ0N0cmwiOiAxLjgsICJNdWx0aUxpbmVUZXh0IjogIlNXSVRDSCIsICJQYWRkaW5nQm90dG9tQ3RybCI6IDIuMCwgIlBhZGRpbmdMZWZ0Q3RybCI6IDIuMCwgIlBhZGRpbmdSaWdodEN0cmwiOiAyLjAsICJQYWRkaW5nVG9wQ3RybCI6IDIuMCwgIldpZHRoQ3RybCI6IDEuMywgImFkdmFuY2VkQ2hlY2tib3giOiBmYWxzZSwgImlubGluZUZvcm1hdFRleHRib3giOiBmYWxzZSwgImxpbmVvdmVyU3R5bGVDaG9pY2UiOiAiU3F1YXJlIiwgImxpbmVvdmVyVGhpY2tuZXNzQ3RybCI6IDF9")
@@
 		(tags "FSM101 ")
 		(property "Reference" "SW2"
-			(at 8.8 -4.6 0)
+			(at 8.8 -3 0)
 			(unlocked yes)
 			(layer "F.SilkS")
@@
 		)
 		(fp_circle
-			(center -7.8994 -2.5)
-			(end -7.6962 -2.5)
+			(center -6.65 -0.85)
+			(end -6.4468 -0.85)
 			(stroke
 				(width 0.1524)
 				(type solid)
 			)
-			(fill no)
+			(fill yes)
 			(layer "F.SilkS")
 		)
@@
 		(tags "FSM101 ")
 		(property "Reference" "SW3"
-			(at -8.8 -4.7 0)
+			(at -8.8 2.9 0)
 			(unlocked yes)
 			(layer "F.SilkS")
@@
 		)
 		(fp_circle
-			(center -7.8994 -2.5)
-			(end -7.6962 -2.5)
+			(center -6.65 -0.85)
+			(end -6.4468 -0.85)
 			(stroke
 				(width 0.1524)
 				(type solid)
 			)
-			(fill no)
+			(fill yes)
 			(layer "F.SilkS")
 		)
@@
 		(layer "Edge.Cuts")
 	)
-	(gr_line
-		(start 53 105)
-		(end 58 105)
-		(stroke
-			(width 0.1)
-			(type solid)
-		)
-		(layer "Edge.Cuts")
-	)
 	(gr_arc
 		(start 105 131)
@@
 	)
 	(gr_line
-		(start 82 105)
-		(end 87 105)
-		(stroke
-			(width 0.1)
-			(type solid)
-		)
-		(layer "Edge.Cuts")
-	)
-	(gr_line
 		(start 82 132)
 		(end 58 132)
@@
 	)
 	(gr_line
+		(start 87 105)
+		(end 82 105)
+		(stroke
+			(width 0.1)
+			(type solid)
+		)
+		(layer "Edge.Cuts")
+	)
+	(gr_line
 		(start 107.1 112.5)
 		(end 105 112.5)
@@
 		(layer "Edge.Cuts")
 	)
+	(gr_line
+		(start 53 105)
+		(end 58 105)
+		(stroke
+			(width 0.1)
+			(type solid)
+		)
+		(layer "Edge.Cuts")
+	)
 	(gr_text "Maker's Asylum\nTheThing_v7"
 		(at 70 131.468 0)
@@
 		(net_name "/Add_on_Board/GND")
 		(layer "B.Cu")
-		(name "GND")
+		(name "GND_ADDON")
 		(hatch edge 0.5)
-		(priority 1)
 		(connect_pads
 			(clearance 0.25)
@@
 			(thermal_bridge_width 0.5)
 			(smoothing fillet)
-			(radius 0.508)
+			(radius 0.5)
 		)
 		(polygon
