File: hardware_PCB/TheThing_v7/add_on_board.kicad_sch (KiCad schematic)
At the start: 14 parts, among them J15 HC-SR04, J16 Conn_01x10, Q1 PN2222ABU, SW2 ON, SW3 ON

Commit message: v7 prototype files for PCB and enclosure
Parts:
- R7: value 1k -> 100E
Changed lines of the file:
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@@
 			)
 		)
-		(property "Value" "1k"
+		(property "Value" "100E"
 			(at 163.83 123.19 90)
 			(effects
